File: kicad/ckt-irsense-split/ckt-irsense-split.kicad_pcb (KiCad board)
At the start: 2 copper layers, 50.8 x 25.4 mm, 26 parts, among them J1 SM04B-SRSS, J2 SM04B-SRSS, J3 SM04B-SRSS, J4 SM04B-SRSS, Q1 SSM6N357R, U1 AP7381-33Y, U2 LTV-357T, U3 LTV-357T

Commit message: Updates after reviewing
Other:
- board text added: "(ISO)"
- board text added: "OUT 1"
- board text added: "SENSOR IN"
- board text removed: "MAIN BOARD"
- board text removed: "SENSOR"
Changed lines of the file:
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@@
 	)
 	(gr_text "PWR"
-		(at 44.704 37.338 0)
+		(at 44.704 37.084 0)
 		(layer "F.SilkS")
 		(effects
@@
 		)
 	)
-	(gr_text "MAIN\nBOARD"
-		(at 38.1 34.036 0)
+	(gr_text "(ISO)"
+		(at 55.118 34.036 0)
+		(layer "F.SilkS")
+		(effects
+			(font
+				(size 1.016 1.016)
+				(thickness 0.2032)
+			)
+			(justify top)
+		)
+	)
+	(gr_text "(ISO)"
+		(at 63.5 34.036 0)
+		(layer "F.SilkS")
+		(effects
+			(font
+				(size 1.016 1.016)
+				(thickness 0.2032)
+			)
+			(justify top)
+		)
+	)
+	(gr_text "OUT 1"
+		(at 38.1 32.131 0)
 		(layer "F.SilkS")
 		(effects
@@
 				(thickness 0.2032)
 			)
+			(justify top)
 		)
 	)
-	(gr_text "SENSOR"
-		(at 46.482 33.02 0)
+	(gr_text "SENSOR\nIN"
+		(at 46.482 32.131 0)
 		(layer "F.SilkS")
 		(effects
@@
 				(thickness 0.2032)
 			)
+			(justify top)
 		)
 	)
 	(gr_text "OUT 2"
-		(at 55.118 33.02 0)
+		(at 55.118 32.131 0)
 		(layer "F.SilkS")
 		(effects
@@
 				(thickness 0.2032)
 			)
+			(justify top)
 		)
 	)
 	(gr_text "OUT 3"
-		(at 63.5 33.02 0)
+		(at 63.5 32.131 0)
 		(layer "F.SilkS")
 		(effects
@@
 				(thickness 0.2032)
 			)
+			(justify top)
 		)
 	)
