File: kicad/ckt-irsense-tiny2pc/ckt-irsense-tiny2pc.kicad_pcb (KiCad board)
At the start: 2 copper layers, 38.1 x 12.7 mm, 17 parts, among them J1 SM04B-SRSS, J11 Conn_AVR_TagConnect_TC2030, J3 SM04B-SRSS, Q1 SSM6N357R, U1 AP7381-33Y, U2 ATtiny13A-SS

Commit message: Minor ckt-irsense-tiny2pc updates
Other:
- board text added: "CKT-IRSENSE-TINY2PC v1.0 iascaled.com ©2026"
- board text removed: "CKT-IRSENSE-TINY2PC iascaled.com ©2026"
Changed lines of the file:
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@@
 		)
 	)
-	(gr_text "CKT-IRSENSE-TINY2PC\niascaled.com ©2026"
-		(at 52.197 27.305 -0)
+	(gr_text "CKT-IRSENSE-TINY2PC v1.0\niascaled.com ©2026"
+		(at 61 27.5 0)
 		(layer "B.SilkS")
 		(effects
@@
 				(thickness 0.1524)
 			)
-			(justify mirror)
+			(justify left mirror)
 		)
 	)
